File: ESP32-Radio.sch (KiCad schematic (older format))
At the start: 71 parts, among them J1 BNC, J11 Conn_01x04_Female, J2 Audio_Jack, J3 Pad, J4 Pad, J6 Audio_Jack, J8 PCB_SMA, T1 6:31, T2 31:6, T3 T50_SPLITTER, T4 T50_SPLITTER, U1 LM358, U10 si5351, U11 LD33V, U2 LM358, U3 LM358, U6 MCP1703A-2502_SOT223, U7 FST3253, U9 LM358

Commit message: fixed references
Parts:
- C22, C23, C24, C25: symbol IQ-Tayloe-Mixer-rescue:1.0UF-0805-25V-(+80_-20%)-phase_v3-eagle-import -> Xenir:Capacitor
- C30: symbol IQ-Tayloe-Mixer-rescue:C5_3.5-Tayloe_Detector_v5-eagle-import -> ESP32-Radio-rescue:C5_3.5-Tayloe_Detector_v5-eagle-import-IQ-Tayloe-Mixer-rescue
- R1, R11, R12, R13, R14, R2, R3: symbol IQ-Tayloe-Mixer-rescue:0.3OHM-0805-1_8W-1%-phase_v3-eagle-import -> Xenir:Resistor
- R4: symbol IQ-Tayloe-Mixer-rescue:0.3OHM-0805-1_8W-1%-phase_v3-eagle-import -> ESP32-Radio-rescue:0.3OHM-0805-1_8W-1%-phase_v3-eagle-import-IQ-Tayloe-Mixer-rescue
- U$1: symbol IQ-Tayloe-Mixer-rescue:FST3253-Tayloe_Detector_v5-eagle-import -> Xenir:FST3253
Changed lines of the file:
@@
 	8350 7500 8350 6600
 $Comp
-L IQ-Tayloe-Mixer-rescue:GND-Tayloe_Detector_v5-eagle-import #GND01
+L ESP32-Radio-rescue:GND-Tayloe_Detector_v5-eagle-import-IQ-Tayloe-Mixer-rescue #GND01
 U 1 1 12C122FD
 P 8750 6400
@@
 $EndComp
 $Comp
-L IQ-Tayloe-Mixer-rescue:C5_3.5-Tayloe_Detector_v5-eagle-import C30
+L ESP32-Radio-rescue:C5_3.5-Tayloe_Detector_v5-eagle-import-IQ-Tayloe-Mixer-rescue C30
 U 1 1 5EE9C731
 P 9450 5200
@@
 	4550 5600 4550 5200
 $Comp
-L IQ-Tayloe-Mixer-rescue:0.3OHM-0805-1_8W-1%-phase_v3-eagle-import R1
+L Xenir:Resistor R1
 U 1 1 5EF82F89
 P 2150 5200
@@
 $EndComp
 $Comp
-L IQ-Tayloe-Mixer-rescue:0.3OHM-0805-1_8W-1%-phase_v3-eagle-import R3
+L Xenir:Resistor R3
 U 1 1 5EF82F8F
 P 2550 5600
@@
 $EndComp
 $Comp
-L IQ-Tayloe-Mixer-rescue:0.3OHM-0805-1_8W-1%-phase_v3-eagle-import R11
+L Xenir:Resistor R11
 U 1 1 5EF82F95
 P 4350 5200
@@
 $EndComp
 $Comp
-L IQ-Tayloe-Mixer-rescue:0.3OHM-0805-1_8W-1%-phase_v3-eagle-import R13
+L Xenir:Resistor R13
 U 1 1 5EF82F9B
 P 4750 5600
@@
 $EndComp
 $Comp
-L IQ-Tayloe-Mixer-rescue:0.3OHM-0805-1_8W-1%-phase_v3-eagle-import R2
+L Xenir:Resistor R2
 U 1 1 5EF82FC5
 P 2150 6700
@@
 $EndComp
 $Comp
-L IQ-Tayloe-Mixer-rescue:0.3OHM-0805-1_8W-1%-phase_v3-eagle-import R4
+L ESP32-Radio-rescue:0.3OHM-0805-1_8W-1%-phase_v3-eagle-import-IQ-Tayloe-Mixer-rescue R4
 U 1 1 5EF82FCB
 P 2550 7100
@@
 $EndComp
 $Comp
-L IQ-Tayloe-Mixer-rescue:0.3OHM-0805-1_8W-1%-phase_v3-eagle-import R12
+L Xenir:Resistor R12
 U 1 1 5EF82FD1
 P 4350 6700
@@
 $EndComp
 $Comp
-L IQ-Tayloe-Mixer-rescue:0.3OHM-0805-1_8W-1%-phase_v3-eagle-import R14
+L Xenir:Resistor R14
 U 1 1 5EF82FD7
 P 4750 7100
@@
 	8750 6100 8750 6300
 $Comp
-L IQ-Tayloe-Mixer-rescue:FST3253-Tayloe_Detector_v5-eagle-import U$1
+L Xenir:FST3253 U$1
 U 1 1 6E1B97F5
-P 11550 6300
-F 0 "U$1" H 8950 7025 59  0000 L BNN
-F 1 "FST3253" H 8950 5600 59  0000 L BNN
-F 2 "Xenir:SO16" H 11550 6300 50  0001 C CNN
-F 3 "" H 11550 6300 50  0001 C CNN
-	1    11550 6300
+P 9900 4950
+F 0 "U$1" H 7300 5675 59  0000 L BNN
+F 1 "FST3253" H 7300 4250 59  0000 L BNN
+F 2 "Xenir:SO16" H 9900 4950 50  0001 C CNN
+F 3 "" H 9900 4950 50  0001 C CNN
+	1    9900 4950
 	1    0    0    -1
 $EndComp
@@
 $EndComp
 $Comp
-L IQ-Tayloe-Mixer-rescue:1.0UF-0805-25V-(+80_-20%)-phase_v3-eagle-import C22
+L Xenir:Capacitor C22
 U 1 1 5EEBD3D7
-P 7100 6050
-F 0 "C22" H 7160 6165 70  0000 L BNN
-F 1 ".022uF" H 7160 5965 70  0000 L BNN
-F 2 "Xenir:Capacitor 1206" H 7100 6050 50  0001 C CNN
-F 3 "" H 7100 6050 50  0001 C CNN
-	1    7100 6050
-	1    0    0    -1
+P 7100 6000
+F 0 "C22" H 6950 5700 70  0000 L BNN
+F 1 ".022uF" H 6850 5800 70  0000 L BNN
+F 2 "Xenir:Capacitor 1206" H 7100 6000 50  0001 C CNN
+F 3 "" H 7100 6000 50  0001 C CNN
+	1    7100 6000
+	0    -1   -1   0
 $EndComp
 $Comp
@@
 $EndComp
 $Comp
-L IQ-Tayloe-Mixer-rescue:1.0UF-0805-25V-(+80_-20%)-phase_v3-eagle-import C23
+L Xenir:Capacitor C23
 U 1 1 5EEBE874
-P 7100 6500
-F 0 "C23" H 7160 6615 70  0000 L BNN
-F 1 ".022uF" H 7160 6415 70  0000 L BNN
-F 2 "Xenir:Capacitor 1206" H 7100 6500 50  0001 C CNN
-F 3 "" H 7100 6500 50  0001 C CNN
-	1    7100 6500
-	1    0    0    -1
+P 7100 6450
+F 0 "C23" H 7050 6700 70  0000 L BNN
+F 1 ".022uF" H 7000 6600 70  0000 L BNN
+F 2 "Xenir:Capacitor 1206" H 7100 6450 50  0001 C CNN
+F 3 "" H 7100 6450 50  0001 C CNN
+	1    7100 6450
+	0    1    1    0
 $EndComp
 $Comp
@@
 $EndComp
 $Comp
-L IQ-Tayloe-Mixer-rescue:1.0UF-0805-25V-(+80_-20%)-phase_v3-eagle-import C24
+L Xenir:Capacitor C24
 U 1 1 5EED34B4
-P 7100 6950
-F 0 "C24" H 7160 7065 70  0000 L BNN
-F 1 ".022uF" H 7160 6865 70  0000 L BNN
-F 2 "Xenir:Capacitor 1206" H 7100 6950 50  0001 C CNN
-F 3 "" H 7100 6950 50  0001 C CNN
-	1    7100 6950
-	1    0    0    -1
+P 7100 6900
+F 0 "C24" H 7050 7150 70  0000 L BNN
+F 1 ".022uF" H 7000 7050 70  0000 L BNN
+F 2 "Xenir:Capacitor 1206" H 7100 6900 50  0001 C CNN
+F 3 "" H 7100 6900 50  0001 C CNN
+	1    7100 6900
+	0    1    1    0
 $EndComp
 $Comp
@@
 $EndComp
 $Comp
-L IQ-Tayloe-Mixer-rescue:1.0UF-0805-25V-(+80_-20%)-phase_v3-eagle-import C25
+L Xenir:Capacitor C25
 U 1 1 5EED8105
-P 7100 7400
-F 0 "C25" H 7160 7515 70  0000 L BNN
-F 1 ".022uF" H 7160 7315 70  0000 L BNN
-F 2 "Xenir:Capacitor 1206" H 7100 7400 50  0001 C CNN
-F 3 "" H 7100 7400 50  0001 C CNN
-	1    7100 7400
-	1    0    0    -1
+P 7100 7350
+F 0 "C25" H 6950 7050 70  0000 L BNN
+F 1 ".022uF" H 6850 7150 70  0000 L BNN
+F 2 "Xenir:Capacitor 1206" H 7100 7350 50  0001 C CNN
+F 3 "" H 7100 7350 50  0001 C CNN
+	1    7100 7350
+	0    -1   -1   0
 $EndComp
 $Comp
@@
 Wire Wire Line
 	7800 6800 8150 6800
-Connection ~ 7100 5850
 Connection ~ 8150 6800
 Wire Wire Line
@@
 Wire Wire Line
 	8050 6500 8550 6500
-Connection ~ 7100 6300
 Connection ~ 8550 6500
 Wire Wire Line
@@
 Wire Wire Line
 	7600 6700 8250 6700
-Connection ~ 7100 6750
 Connection ~ 8250 6700
 Wire Wire Line
@@
 Text GLabel 10150 6000 2    50   Input ~ 0
 LO_90
+Connection ~ 7100 6300
+Connection ~ 7100 5850
+Connection ~ 7100 6750
 $EndSCHEMATC

Commit message: more fixes
Parts:
- removed C29: .1uF, Xenir:Capacitor 1206, symbol Xenir:Capacitor
- removed U9: LM358, Xenir:SOIC8, symbol Xenir:LM358
- C30: symbol ESP32-Radio-rescue:C5_3.5-Tayloe_Detector_v5-eagle-import-IQ-Tayloe-Mixer-rescue -> Xenir:Capacitor
- U2: footprint Xenir:SOIC8 -> Xenir:SO08
- U3: footprint Xenir:SO08 -> Xenir:SOIC8
- renumbered U$1 to U8
Changed lines of the file:
@@
 $EndComp
 $Comp
-L ESP32-Radio-rescue:C5_3.5-Tayloe_Detector_v5-eagle-import-IQ-Tayloe-Mixer-rescue C30
+L Xenir:Capacitor C30
 U 1 1 5EE9C731
-P 9450 5200
-F 0 "C30" H 9510 5215 59  0000 L BNN
-F 1 ".1uF" H 9510 5015 59  0000 L BNN
-F 2 "Xenir:Capacitor 0805" H 9450 5200 50  0001 C CNN
-F 3 "" H 9450 5200 50  0001 C CNN
-	1    9450 5200
-	1    0    0    -1
+P 9450 5250
+F 0 "C30" H 9350 5350 59  0000 L BNN
+F 1 ".1uF" H 9350 5100 59  0000 L BNN
+F 2 "Xenir:Capacitor 0805" H 9450 5250 50  0001 C CNN
+F 3 "" H 9450 5250 50  0001 C CNN
+	1    9450 5250
+	0    1    1    0
 $EndComp
 $Comp
@@
 U 1 1 5EF82F89
 P 2150 5200
-F 0 "R1" H 2150 5260 70  0000 C BNN
-F 1 "10k" H 2150 5140 70  0000 C TNN
+F 0 "R1" H 2150 5260 28  0000 C BNN
+F 1 "10k" H 2150 5140 28  0000 C TNN
 F 2 "Xenir:Resistor 0805" H 2150 5200 50  0001 C CNN
 F 3 "" H 2150 5200 50  0001 C CNN
@@
 U 1 1 5EF82F8F
 P 2550 5600
-F 0 "R3" H 2550 5660 70  0000 C BNN
-F 1 "10k" H 2550 5540 70  0000 C TNN
+F 0 "R3" H 2550 5660 28  0000 C BNN
+F 1 "10k" H 2550 5540 28  0000 C TNN
 F 2 "Xenir:Resistor 0805" H 2550 5600 50  0001 C CNN
 F 3 "" H 2550 5600 50  0001 C CNN
@@
 U 1 1 5EF82F95
 P 4350 5200
-F 0 "R11" H 4350 5260 70  0000 C BNN
-F 1 "10k" H 4350 5140 70  0000 C TNN
+F 0 "R11" H 4350 5260 28  0000 C BNN
+F 1 "10k" H 4350 5140 28  0000 C TNN
 F 2 "Xenir:Resistor 0805" H 4350 5200 50  0001 C CNN
 F 3 "" H 4350 5200 50  0001 C CNN
@@
 U 1 1 5EF82F9B
 P 4750 5600
-F 0 "R13" H 4750 5660 70  0000 C BNN
-F 1 "10k" H 4750 5540 70  0000 C TNN
+F 0 "R13" H 4750 5660 28  0000 C BNN
+F 1 "10k" H 4750 5540 28  0000 C TNN
 F 2 "Xenir:Resistor 0805" H 4750 5600 50  0001 C CNN
 F 3 "" H 4750 5600 50  0001 C CNN
@@
 U 1 1 5EF82FC5
 P 2150 6700
-F 0 "R2" H 2150 6760 70  0000 C BNN
-F 1 "10k" H 2150 6640 70  0000 C TNN
+F 0 "R2" H 2150 6760 28  0000 C BNN
+F 1 "10k" H 2150 6640 28  0000 C TNN
 F 2 "Xenir:Resistor 0805" H 2150 6700 50  0001 C CNN
 F 3 "" H 2150 6700 50  0001 C CNN
@@
 U 1 1 5EF82FCB
 P 2550 7100
-F 0 "R4" H 2550 7160 70  0000 C BNN
-F 1 "10k" H 2550 7040 70  0000 C TNN
+F 0 "R4" H 2550 7160 28  0000 C BNN
+F 1 "10k" H 2550 7040 28  0000 C TNN
 F 2 "Xenir:Resistor 0805" H 2550 7100 50  0001 C CNN
 F 3 "" H 2550 7100 50  0001 C CNN
@@
 U 1 1 5EF82FD1
 P 4350 6700
-F 0 "R12" H 4350 6760 70  0000 C BNN
-F 1 "10k" H 4350 6640 70  0000 C TNN
+F 0 "R12" H 4350 6760 28  0000 C BNN
+F 1 "10k" H 4350 6640 28  0000 C TNN
 F 2 "Xenir:Resistor 0805" H 4350 6700 50  0001 C CNN
 F 3 "" H 4350 6700 50  0001 C CNN
@@
 U 1 1 5EF82FD7
 P 4750 7100
-F 0 "R14" H 4750 7160 70  0000 C BNN
-F 1 "10k" H 4750 7040 70  0000 C TNN
+F 0 "R14" H 4750 7160 28  0000 C BNN
+F 1 "10k" H 4750 7040 28  0000 C TNN
 F 2 "Xenir:Resistor 0805" H 4750 7100 50  0001 C CNN
 F 3 "" H 4750 7100 50  0001 C CNN
@@
 	1    0    0    -1
 $EndComp
-Connection ~ 9450 5400
 Connection ~ 8750 6300
 Wire Wire Line
 	8750 6100 8750 6300
 $Comp
-L Xenir:FST3253 U$1
+L Xenir:FST3253 U8
 U 1 1 6E1B97F5
 P 9900 4950
-F 0 "U$1" H 7300 5675 59  0000 L BNN
-F 1 "FST3253" H 7300 4250 59  0000 L BNN
+F 0 "U8" H 9350 3550 59  0000 L BNN
+F 1 "FST3253" H 9250 3400 59  0000 L BNN
 F 2 "Xenir:SO16" H 9900 4950 50  0001 C CNN
 F 3 "" H 9900 4950 50  0001 C CNN
@@
 U 1 1 5EEBD3D7
 P 7100 6000
-F 0 "C22" H 6950 5700 70  0000 L BNN
-F 1 ".022uF" H 6850 5800 70  0000 L BNN
+F 0 "C22" H 7050 5800 28  0000 L BNN
+F 1 ".022uF" H 7000 5850 28  0000 L BNN
 F 2 "Xenir:Capacitor 1206" H 7100 6000 50  0001 C CNN
 F 3 "" H 7100 6000 50  0001 C CNN
@@
 $EndComp
 $Comp
-L power:GND #PWR022
-U 1 1 5EEBE297
-P 7100 6150
-F 0 "#PWR022" H 7100 5900 50  0001 C CNN
-F 1 "GND" H 7100 6000 50  0000 C CNN
-F 2 "" H 7100 6150 50  0001 C CNN
-F 3 "" H 7100 6150 50  0001 C CNN
-	1    7100 6150
-	1    0    0    -1
-$EndComp
-$Comp
 L Xenir:Capacitor C23
 U 1 1 5EEBE874
 P 7100 6450
-F 0 "C23" H 7050 6700 70  0000 L BNN
-F 1 ".022uF" H 7000 6600 70  0000 L BNN
+F 0 "C23" H 7050 6650 28  0000 L BNN
+F 1 ".022uF" H 7000 6600 28  0000 L BNN
 F 2 "Xenir:Capacitor 1206" H 7100 6450 50  0001 C CNN
 F 3 "" H 7100 6450 50  0001 C CNN
@@
 P 7100 6600
 F 0 "#PWR023" H 7100 6350 50  0001 C CNN
-F 1 "GND" H 7100 6450 50  0000 C CNN
+F 1 "GND" H 7250 6550 50  0000 C CNN
 F 2 "" H 7100 6600 50  0001 C CNN
 F 3 "" H 7100 6600 50  0001 C CNN
@@
 U 1 1 5EED34B4
 P 7100 6900
-F 0 "C24" H 7050 7150 70  0000 L BNN
-F 1 ".022uF" H 7000 7050 70  0000 L BNN
+F 0 "C24" H 7100 7100 28  0000 L BNN
+F 1 ".022uF" H 7050 7050 28  0000 L BNN
 F 2 "Xenir:Capacitor 1206" H 7100 6900 50  0001 C CNN
 F 3 "" H 7100 6900 50  0001 C CNN
@@
 P 7100 7050
 F 0 "#PWR024" H 7100 6800 50  0001 C CNN
-F 1 "GND" H 7100 6900 50  0000 C CNN
+F 1 "GND" H 7250 7000 50  0000 C CNN
 F 2 "" H 7100 7050 50  0001 C CNN
 F 3 "" H 7100 7050 50  0001 C CNN
@@
 U 1 1 5EED8105
 P 7100 7350
-F 0 "C25" H 6950 7050 70  0000 L BNN
-F 1 ".022uF" H 6850 7150 70  0000 L BNN
+F 0 "C25" H 7050 7150 28  0000 L BNN
+F 1 ".022uF" H 7000 7200 28  0000 L BNN
 F 2 "Xenir:Capacitor 1206" H 7100 7350 50  0001 C CNN
 F 3 "" H 7100 7350 50  0001 C CNN
@@
 P 7100 7500
 F 0 "#PWR025" H 7100 7250 50  0001 C CNN
-F 1 "GND" H 7100 7350 50  0000 C CNN
+F 1 "GND" H 7250 7450 50  0000 C CNN
 F 2 "" H 7100 7500 50  0001 C CNN
 F 3 "" H 7100 7500 50  0001 C CNN
@@
 U 3 1 5EAF812F
 P 3000 2750
-F 0 "U1" H 2850 2700 70  0000 L BNN
-F 1 "LM358" H 2950 3000 70  0000 L BNN
+F 0 "U1" H 2850 2700 39  0000 L BNN
+F 1 "LM358" V 2750 2600 70  0000 L BNN
 F 2 "Xenir:SO08" H 2950 2700 50  0001 C CNN
 F 3 "" H 2950 2700 50  0001 C CNN
@@
 U 3 1 5EB0186E
 P 3450 2750
-F 0 "U2" H 3300 2700 70  0000 L BNN
-F 1 "LM358" H 3400 3000 70  0000 L BNN
+F 0 "U2" H 3300 2700 39  0000 L BNN
+F 1 "LM358" V 3200 2600 70  0000 L BNN
 F 2 "Xenir:SO08" H 3400 2700 50  0001 C CNN
 F 3 "" H 3400 2700 50  0001 C CNN
@@
 U 3 1 5EC1C0E9
 P 3850 2750
-F 0 "U3" H 3700 2700 70  0000 L BNN
-F 1 "LM358" H 3800 3000 70  0000 L BNN
+F 0 "U3" H 3700 2700 39  0000 L BNN
+F 1 "LM358" V 3600 2600 70  0000 L BNN
 F 2 "Xenir:SOIC8" H 3800 2700 50  0001 C CNN
 F 3 "" H 3800 2700 50  0001 C CNN
@@
 F 0 "U2" H 4700 6550 70  0000 L BNN
 F 1 "LM358" H 4800 6850 70  0000 L BNN
-F 2 "Xenir:SOIC8" H 4800 6550 50  0001 C CNN
+F 2 "Xenir:SO08" H 4800 6550 50  0001 C CNN
 F 3 "" H 4800 6550 50  0001 C CNN
 	2    4850 6600
@@
 U 1 1 5EA318D2
 P 8700 10200
-F 0 "U7" H 8250 9931 50  0000 C CNN
-F 1 "FST3253" H 8250 9840 50  0000 C CNN
+F 0 "U7" H 8250 8900 50  0000 C CNN
+F 1 "FST3253" H 8250 8800 50  0000 C CNN
 F 2 "Xenir:SO16" H 8600 9600 50  0001 C CNN
 F 3 "" H 8600 9600 50  0001 C CNN
@@
 F 0 "U3" H 3150 12300 70  0000 C CNN
 F 1 "LM358" H 3450 12450 70  0000 C CNN
-F 2 "Xenir:SO08" H 3150 12250 50  0001 C CNN
+F 2 "Xenir:SOIC8" H 3150 12250 50  0001 C CNN
 F 3 "" H 3150 12250 50  0001 C CNN
 	2    3200 12300
 	-1   0    0    -1
 $EndComp
-$Comp
-L Xenir:LM358 U9
-U 3 1 5EAA2951
-P 9750 10250
-F 0 "U9" H 9778 10311 70  0000 L CNN
-F 1 "LM358" H 9778 10190 70  0000 L CNN
-F 2 "Xenir:SOIC8" H 9700 10200 50  0001 C CNN
-F 3 "" H 9700 10200 50  0001 C CNN
-	3    9750 10250
-	1    0    0    -1
-$EndComp
 Wire Wire Line
 	3850 11100 3700 11100
@@
 	3500 12400 3750 12400
 $Comp
-L power:GND #PWR036
-U 1 1 5EAC6CB2
-P 9650 10550
-F 0 "#PWR036" H 9650 10300 50  0001 C CNN
-F 1 "GND" H 9655 10377 50  0000 C CNN
-F 2 "" H 9650 10550 50  0001 C CNN
-F 3 "" H 9650 10550 50  0001 C CNN
-	1    9650 10550
-	1    0    0    -1
-$EndComp
-$Comp
-L power:+12V #PWR035
-U 1 1 5EAC7EBD
-P 9650 9950
-F 0 "#PWR035" H 9650 9800 50  0001 C CNN
-F 1 "+12V" H 9665 10123 50  0000 C CNN
-F 2 "" H 9650 9950 50  0001 C CNN
-F 3 "" H 9650 9950 50  0001 C CNN
-	1    9650 9950
-	1    0    0    -1
-$EndComp
-$Comp
-L Xenir:Capacitor C29
-U 1 1 5EAC8FB2
-P 9400 10250
-F 0 "C29" H 9200 10400 50  0000 L CNN
-F 1 ".1uF" H 9450 10400 50  0000 L CNN
-F 2 "Xenir:Capacitor 1206" H 9400 10250 50  0001 C CNN
-F 3 "" H 9400 10250 50  0001 C CNN
-	1    9400 10250
-	0    -1   -1   0
-$EndComp
-Wire Wire Line
-	9400 10100 9400 9950
-Wire Wire Line
-	9400 9950 9650 9950
-Connection ~ 9650 9950
-Wire Wire Line
-	9650 10550 9400 10550
-Wire Wire Line
-	9400 10550 9400 10400
-Connection ~ 9650 10550
-$Comp
 L Device:R_Small_US R5
 U 1 1 5EADA2EC
@@
 Connection ~ 5450 1400
 $Comp
-L power:+2V5 #PWR?
+L power:+2V5 #PWR0101
 U 1 1 6100363A
 P 7450 9350
-F 0 "#PWR?" H 7450 9200 50  0001 C CNN
+F 0 "#PWR0101" H 7450 9200 50  0001 C CNN
 F 1 "+2V5" H 7465 9523 50  0000 C CNN
 F 2 "" H 7450 9350 50  0001 C CNN
@@
 Connection ~ 7100 5850
 Connection ~ 7100 6750
+Connection ~ 9450 5400
+$Comp
+L power:GND #PWR022
+U 1 1 5EEBE297
+P 7100 6150
+F 0 "#PWR022" H 7100 5900 50  0001 C CNN
+F 1 "GND" H 7250 6100 50  0000 C CNN
+F 2 "" H 7100 6150 50  0001 C CNN
+F 3 "" H 7100 6150 50  0001 C CNN
+	1    7100 6150
+	1    0    0    -1
+$EndComp
 $EndSCHEMATC
